File: hardware/sailface-mega-shield-v0.3/sailface-mega-shield.kicad_pcb (KiCad board)
At the start: 2 copper layers, 101.6 x 53.3 mm, 35 parts, among them P1 Digital, P10 CONN_01X01, P11 CONN_01X01, P12 CONN_01X01, P13 CONN_01X01, P2 Power, P3 Analog, P4 Analog, P5 PWM, P6 PWM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

Commit message: circuit board.
Parts:
- removed ARDUINO_POWER1: ARDUINO_POWER, Connector_PinSocket_2.54mm:PinSocket_1x02_P2.54mm_Vertical
- added P11: CONN_01X01, Socket_Arduino_Mega:Arduino_1pin, F.Cu at (109.2, 106.2)
- MOTOR_PWM: renamed from MOTOR_PWM_PORT1; footprint Connector_PinSocket_2.54mm:PinSocket_1x01_P2.54mm_Vertical -> Connector_PinSocket_2.54mm:PinSocket_1x02_P2.54mm_Vertical
- R2, R3, R4, R5, R6: footprint Resistor_THT:R_Axial_DIN0204_L3.6mm_D1.6mm_P2.54mm_Vertical -> Resistor_THT:R_Axial_DIN0204_L3.6mm_D1.6mm_P7.62mm_Horizontal
- moved R3 4.58 mm to (151.1, 88.9), turned to 180 degrees
- moved R4 1.27 mm to (144.8, 108.0)
- turned MOTOR_PWM to 0 degrees
- renumbered MOTOR_POWER1 to MOTOR
Connections:
- P2 pad 8: /Vin -> +12V
Routing:
- net /IRIDIUM_ON: track 46.8 -> 39.2 mm
- net GND: track 250.6 -> 246.3 mm
- net /MPU_ON: track 23.6 -> 19.5 mm
- net Net-(MPU_TOGGLE1-Pad2): track 10.0 -> 14.0 mm
- net Net-(BLUETOOTH1-Pad3): track 18.3 -> 22.0 mm
- net /MOTOR_PWM: track 124.3 -> 127.7 mm
- net +12V: track 118.4 -> 121.8 mm
- net +3V3: track 138.6 -> 136.4 mm
- net /BAT_VOLTAGE_MONITOR: track 19.9 -> 21.7 mm
- net +5V: track 118.7 -> 119.8 mm
- net /BLUETOOTH_ON: track 26.5 -> 25.4 mm
- net /BATTERY_IN: track 62.7 -> 62.0 mm
