File: hardware/sailface-mega-shield-v0.3/sailface-mega-shield.kicad_sch (KiCad schematic)
At the start: 35 parts, among them P1 Digital, P10 CONN_01X01, P11 CONN_01X01, P12 CONN_01X01, P13 CONN_01X01, P2 Power, P3 Analog, P4 Analog, P5 PWM, P6 PWM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

Commit message: circuit board.
Parts:
- removed ARDUINO_POWER1: ARDUINO_POWER, Connector_PinSocket_2.54mm:PinSocket_1x02_P2.54mm_Vertical, symbol Connector:Screw_Terminal_01x02
- MOTOR_PWM_PORT1: value MOTOR_PWM_PORT -> (none); footprint Connector_PinSocket_2.54mm:PinSocket_1x01_P2.54mm_Vertical -> (none); symbol Connector_Generic:Conn_01x01 -> Connector_Generic:Conn_01x02
- R2, R3, R4, R6: value 1K -> (none); footprint Resistor_THT:R_Axial_DIN0204_L3.6mm_D1.6mm_P2.54mm_Vertical -> (none)
- R5: value 4.7K -> (none); footprint Resistor_THT:R_Axial_DIN0204_L3.6mm_D1.6mm_P2.54mm_Vertical -> (none)
Connections:
- net Vin is gone; now on net +12V: P2.8 (Pin_8)
- net GND: now also MOTOR_PWM_PORT1.2 (Pin_2)
