File: schematics/sailboard-esp/Power.kicad_sch (KiCad schematic)
At the start: 15 parts

Commit message: v1.1 of sailboard.
Parts:
- added CURRENT_SOLAR1: INA219BxD, Package_SO:SOIC-8_3.9x4.9mm_P1.27mm, symbol Analog_ADC:INA219BxD
- added R_SHUNT2: 100mOhms, Resistor_SMD:R_2512_6332Metric, symbol Device:R
- renumbered CURRENT_SENSOR1 to CURRENT_MAIN1
Connections:
- net +5V: now also CURRENT_SOLAR1.2 (A0), CURRENT_SOLAR1.5 (VS)
- net GND: now also CURRENT_SOLAR1.1 (A1), CURRENT_SOLAR1.6 (GND)
- net SCL: now also CURRENT_SOLAR1.4 (SCL)
- net SDA: now also CURRENT_SOLAR1.3 (SDA)
- new net Battery Charge Pos: CURRENT_SOLAR1.7 (IN-), R_SHUNT2.2
- new net Solar Pos: CURRENT_SOLAR1.8 (IN+), R_SHUNT2.1
Other:
- note added: "A1 GND & A0 +5V equal I2C address = 0x41"

Commit message: version 1.1.
Connections:
- net +5V renamed +5V Output
- net +5V Output: no longer CURRENT_MAIN1.5 (VS), CURRENT_SOLAR1.2 (A0), CURRENT_SOLAR1.5 (VS)
- new net +3.3V: CURRENT_MAIN1.5 (VS), CURRENT_SOLAR1.2 (A0), CURRENT_SOLAR1.5 (VS)
Changed lines of the file:
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@@
   (junction (at 231.14 114.3) (diameter 0) (color 0 0 0 0)
-  )
-  (junction (at 256.54 54.61) (diameter 0) (color 0 0 0 0)
   )
   (junction (at 201.93 81.28) (diameter 0) (color 0 0 0 0)
@@
     (stroke (width 0) (type default) (color 0 0 0 0))
   )
-  (wire (pts (xy 256.54 54.61) (xy 259.08 54.61))
+  (wire (pts (xy 248.92 54.61) (xy 259.08 54.61))
     (stroke (width 0) (type default) (color 0 0 0 0))
   )
@@
     (stroke (width 0) (type default) (color 0 0 0 0))
   )
-  (wire (pts (xy 256.54 49.53) (xy 256.54 54.61))
-    (stroke (width 0) (type default) (color 0 0 0 0))
-  )
   (wire (pts (xy 201.93 134.62) (xy 201.93 137.16))
     (stroke (width 0) (type default) (color 0 0 0 0))
@@
     (stroke (width 0) (type default) (color 0 0 0 0))
   )
-  (wire (pts (xy 248.92 54.61) (xy 256.54 54.61))
-    (stroke (width 0) (type default) (color 0 0 0 0))
-  )
   (wire (pts (xy 62.23 119.38) (xy 68.58 119.38))
     (stroke (width 0) (type default) (color 0 0 0 0))
@@
     (stroke (width 0) (type default) (color 0 0 0 0))
   )
-  (wire (pts (xy 88.9 116.84) (xy 95.25 116.84))
+  (wire (pts (xy 88.9 116.84) (xy 96.52 116.84))
     (stroke (width 0) (type default) (color 0 0 0 0))
   )
@@
     (pin "1")
   )
-  (symbol (lib_id "power:+5V") (at 106.68 40.64 0) (unit 1)
-    (in_bom yes) (on_board yes) (fields_autoplaced)
-    (property "Reference" "#PWR0148" (id 0) (at 106.68 44.45 0)
-      (effects (font (size 1.27 1.27)) hide)
-    )
-    (property "Value" "+5V" (id 1) (at 106.68 35.56 0))
-    (property "Footprint" "" (id 2) (at 106.68 40.64 0)
-      (effects (font (size 1.27 1.27)) hide)
-    )
-    (property "Datasheet" "" (id 3) (at 106.68 40.64 0)
-      (effects (font (size 1.27 1.27)) hide)
-    )
-    (pin "1")
-  )
   (symbol (lib_id "Device:R_Small_US") (at 231.14 57.15 0) (unit 1)
     (in_bom yes) (on_board yes) (fields_autoplaced)
@@
     (pin "8")
   )
-  (symbol (lib_id "power:+5V") (at 256.54 49.53 0) (unit 1)
-    (in_bom yes) (on_board yes) (fields_autoplaced)
-    (property "Reference" "#PWR0109" (id 0) (at 256.54 53.34 0)
-      (effects (font (size 1.27 1.27)) hide)
-    )
-    (property "Value" "+5V" (id 1) (at 256.54 44.45 0))
-    (property "Footprint" "" (id 2) (at 256.54 49.53 0)
-      (effects (font (size 1.27 1.27)) hide)
-    )
-    (property "Datasheet" "" (id 3) (at 256.54 49.53 0)
-      (effects (font (size 1.27 1.27)) hide)
-    )
-    (pin "1")
-  )
   (symbol (lib_id "power:GND") (at 201.93 83.82 0) (unit 1)
     (in_bom yes) (on_board yes) (fields_autoplaced)
@@
     )
     (property "Datasheet" "" (id 3) (at 201.93 83.82 0)
+      (effects (font (size 1.27 1.27)) hide)
+    )
+    (pin "1")
+  )
+  (symbol (lib_id "power:+3.3V") (at 96.52 116.84 270) (unit 1)
+    (in_bom yes) (on_board yes) (fields_autoplaced)
+    (property "Reference" "#PWR0150" (id 0) (at 92.71 116.84 0)
+      (effects (font (size 1.27 1.27)) hide)
+    )
+    (property "Value" "+3.3V" (id 1) (at 100.33 116.8399 90)
+      (effects (font (size 1.27 1.27)) (justify left))
+    )
+    (property "Footprint" "" (id 2) (at 96.52 116.84 0)
+      (effects (font (size 1.27 1.27)) hide)
+    )
+    (property "Datasheet" "" (id 3) (at 96.52 116.84 0)
       (effects (font (size 1.27 1.27)) hide)
     )
@@
     (pin "2")
   )
-  (symbol (lib_id "power:+5V") (at 78.74 91.44 0) (unit 1)
-    (in_bom yes) (on_board yes) (fields_autoplaced)
-    (property "Reference" "#PWR0152" (id 0) (at 78.74 95.25 0)
-      (effects (font (size 1.27 1.27)) hide)
-    )
-    (property "Value" "+5V" (id 1) (at 78.74 86.36 0))
-    (property "Footprint" "" (id 2) (at 78.74 91.44 0)
-      (effects (font (size 1.27 1.27)) hide)
-    )
-    (property "Datasheet" "" (id 3) (at 78.74 91.44 0)
-      (effects (font (size 1.27 1.27)) hide)
-    )
-    (pin "1")
-  )
   (symbol (lib_id "power:GND") (at 165.1 113.03 0) (unit 1)
     (in_bom yes) (on_board yes) (fields_autoplaced)
@@
     )
     (property "Datasheet" "" (id 3) (at 95.25 114.3 0)
+      (effects (font (size 1.27 1.27)) hide)
+    )
+    (pin "1")
+  )
+  (symbol (lib_id "power:+3.3V") (at 78.74 91.44 0) (unit 1)
+    (in_bom yes) (on_board yes) (fields_autoplaced)
+    (property "Reference" "#PWR0148" (id 0) (at 78.74 95.25 0)
+      (effects (font (size 1.27 1.27)) hide)
+    )
+    (property "Value" "+3.3V" (id 1) (at 78.74 86.36 0))
+    (property "Footprint" "" (id 2) (at 78.74 91.44 0)
+      (effects (font (size 1.27 1.27)) hide)
+    )
+    (property "Datasheet" "" (id 3) (at 78.74 91.44 0)
       (effects (font (size 1.27 1.27)) hide)
     )
@@
     (pin "9")
   )
-  (symbol (lib_id "power:+5V") (at 95.25 116.84 270) (unit 1)
-    (in_bom yes) (on_board yes) (fields_autoplaced)
-    (property "Reference" "#PWR0150" (id 0) (at 91.44 116.84 0)
-      (effects (font (size 1.27 1.27)) hide)
-    )
-    (property "Value" "+5V" (id 1) (at 99.06 116.8399 90)
-      (effects (font (size 1.27 1.27)) (justify left))
-    )
-    (property "Footprint" "" (id 2) (at 95.25 116.84 0)
-      (effects (font (size 1.27 1.27)) hide)
-    )
-    (property "Datasheet" "" (id 3) (at 95.25 116.84 0)
-      (effects (font (size 1.27 1.27)) hide)
-    )
-    (pin "1")
-  )
   (symbol (lib_id "power:GND") (at 167.64 62.23 0) (unit 1)
     (in_bom yes) (on_board yes) (fields_autoplaced)
@@
     (pin "2")
   )
+  (symbol (lib_id "power:+3.3V") (at 106.68 40.64 0) (unit 1)
+    (in_bom yes) (on_board yes) (fields_autoplaced)
+    (property "Reference" "#PWR0109" (id 0) (at 106.68 44.45 0)
+      (effects (font (size 1.27 1.27)) hide)
+    )
+    (property "Value" "+3.3V" (id 1) (at 106.68 35.56 0))
+    (property "Footprint" "" (id 2) (at 106.68 40.64 0)
+      (effects (font (size 1.27 1.27)) hide)
+    )
+    (property "Datasheet" "" (id 3) (at 106.68 40.64 0)
+      (effects (font (size 1.27 1.27)) hide)
+    )
+    (pin "1")
+  )
   (symbol (lib_id "Device:R_Small_US") (at 176.53 106.68 0) (unit 1)

Commit message: add capacitor footprint.
Parts:
- C1, C2, C3, C4: footprint (none) -> Capacitor_SMD:C_0603_1608Metric_Pad1.08x0.95mm_HandSolder
Changed lines of the file:
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@@
       (effects (font (size 1.27 1.27)) (justify left))
     )
-    (property "Footprint" "" (id 2) (at 165.1 106.68 0)
+    (property "Footprint" "Capacitor_SMD:C_0603_1608Metric_Pad1.08x0.95mm_HandSolder" (id 2) (at 165.1 106.68 0)
       (effects (font (size 1.27 1.27)) hide)
     )
@@
       (effects (font (size 1.27 1.27)) (justify left))
     )
-    (property "Footprint" "" (id 2) (at 167.64 58.42 0)
+    (property "Footprint" "Capacitor_SMD:C_0603_1608Metric_Pad1.08x0.95mm_HandSolder" (id 2) (at 167.64 58.42 0)
       (effects (font (size 1.27 1.27)) hide)
     )
@@
       (effects (font (size 1.27 1.27)) (justify left))
     )
-    (property "Footprint" "" (id 2) (at 248.92 114.3 0)
+    (property "Footprint" "Capacitor_SMD:C_0603_1608Metric_Pad1.08x0.95mm_HandSolder" (id 2) (at 248.92 114.3 0)
       (effects (font (size 1.27 1.27)) hide)
     )
@@
       (effects (font (size 1.27 1.27)) (justify left))
     )
-    (property "Footprint" "" (id 2) (at 248.92 63.5 0)
-      (effects (font (size 1.27 1.27)) hide)
-    )
+    (property "Footprint" "Capacitor_SMD:C_0603_1608Metric_Pad1.08x0.95mm_HandSolder" (id 2) (at 248.92 63.5 0)
+      (effects (font (size 1.27 1.27)) hide)
+    )

Commit message: move to version 1.2.
Parts:
- removed C4: 22uF, Capacitor_SMD:C_0603_1608Metric_Pad1.08x0.95mm_HandSolder, symbol Device:C_Small
- removed R2: 100K, Resistor_SMD:R_0603_1608Metric, symbol Device:R_Small_US
- removed R6: 75K, Resistor_SMD:R_0603_1608Metric, symbol Device:R_Small_US
- removed R7: 24K, Resistor_SMD:R_0603_1608Metric, symbol Device:R_Small_US
- removed Regulator3V1: MPM3610AGQV-P, MPM3610AGQV-P:MPM3620AGQV-P, symbol MPM3610AGQV-P:MPM3610AGQV-P
- added R2: 39K, Resistor_SMD:R_0603_1608Metric, symbol Device:R_US
- added U1: AP2112K-3.3, Package_TO_SOT_SMD:SOT-23-5, symbol Regulator_Linear:AP2112K-3.3
- C1: value 10uF -> 1uF
- R5: value 19.1K -> 19K
Connections:
- net +12V: no longer C1.1
- net +3.3V Output: now also C1.1, U1.5 (VOUT)
- net +5V Output: now also U1.1 (VIN), U1.3 (EN)
- net GND: now also R2.2, U1.2 (GND)
- net at Regulator5V1.18 (AAM): now also R2.1
- no-connect marks 6 -> 3

Commit message: tweaks.
Parts:
- R2: value 39K -> 53.6K
- R5: value 19K -> 19.1K
Changed lines of the file:
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@@
       (effects (font (size 1.27 1.27)) (justify left))
     )
-    (property "Value" "39K" (id 1) (at 184.15 76.1999 0)
+    (property "Value" "53.6K" (id 1) (at 184.15 76.1999 0)
       (effects (font (size 1.27 1.27)) (justify left))
     )
@@
       (effects (font (size 1.27 1.27)) (justify left))
     )
-    (property "Value" "19K" (id 1) (at 233.68 68.5799 0)
+    (property "Value" "19.1K" (id 1) (at 233.68 68.5799 0)
       (effects (font (size 1.27 1.27)) (justify left))
     )
