File: schematics/sailboard-esp/propulsion.kicad_sch (KiCad schematic)
At the start: 3 parts, among them U3 L293D

Commit message: version 1.1.
Parts:
- MOTOR1, MOTOR2: footprint Connector_PinHeader_2.00mm:PinHeader_1x02_P2.00mm_Vertical -> Connector_PinHeader_2.54mm:PinHeader_1x02_P2.54mm_Vertical
Changed lines of the file:
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@@
       (effects (font (size 1.27 1.27)) (justify left))
     )
-    (property "Footprint" "Connector_PinHeader_2.00mm:PinHeader_1x02_P2.00mm_Vertical" (id 2) (at 100.33 85.09 0)
+    (property "Footprint" "Connector_PinHeader_2.54mm:PinHeader_1x02_P2.54mm_Vertical" (id 2) (at 100.33 85.09 0)
       (effects (font (size 1.27 1.27)) hide)
     )
@@
       (effects (font (size 1.27 1.27)) (justify left))
     )
-    (property "Footprint" "Connector_PinHeader_2.00mm:PinHeader_1x02_P2.00mm_Vertical" (id 2) (at 100.33 69.85 0)
+    (property "Footprint" "Connector_PinHeader_2.54mm:PinHeader_1x02_P2.54mm_Vertical" (id 2) (at 100.33 69.85 0)
       (effects (font (size 1.27 1.27)) hide)
     )

Commit message: move to version 1.2.
Parts:
- removed MOTOR2: MOTOR, Connector_PinHeader_2.54mm:PinHeader_1x02_P2.54mm_Vertical, symbol Connector_Generic:Conn_01x02
- removed U3: L293D, Package_DIP:DIP-16_W7.62mm, symbol Driver_Motor:L293D
- added U2: L293D, Package_DIP:DIP-16_W7.62mm, symbol Driver_Motor:L293D
- MOTOR1: footprint Connector_PinHeader_2.54mm:PinHeader_1x02_P2.54mm_Vertical -> Connector_JST:JST_XH_B2B-XH-A_1x02_P2.50mm_Vertical
Connections:
- net +12V: now also U2.8 (VCC2)
- net +5V: now also U2.16 (VCC1)
- net GND: now also U2.12 (GND), U2.13 (GND), U2.4 (GND), U2.5 (GND)
- net MOTOR_DIRECTION_1: now also U2.2 (1A)
- net MOTOR_DIRECTION_2: now also U2.7 (2A)
- net MOTOR_PWM: now also U2.1 (EN1,2)
- net at MOTOR1.1 (Pin_1): now also U2.3 (1Y)
- net at MOTOR1.2 (Pin_2): now also U2.6 (2Y)
- no-connect marks 3 -> 5
Other:
- moved on the sheet: MOTOR1
Changed lines of the file:
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@@
 (kicad_sch (version 20211123) (generator eeschema)
   (paper "A4")
-  (junction (at 74.93 111.76) (diameter 0) (color 0 0 0 0)
+  (junction (at 74.93 113.03) (diameter 0) (color 0 0 0 0)
   )
-  (junction (at 69.85 111.76) (diameter 0) (color 0 0 0 0)
+  (junction (at 72.39 113.03) (diameter 0) (color 0 0 0 0)
   )
-  (junction (at 67.31 111.76) (diameter 0) (color 0 0 0 0)
+  (junction (at 69.85 113.03) (diameter 0) (color 0 0 0 0)
   )
-  (no_connect (at 59.69 85.09))
   (no_connect (at 59.69 90.17))
   (no_connect (at 59.69 95.25))
-  (wire (pts (xy 74.93 105.41) (xy 74.93 111.76))
+  (no_connect (at 85.09 90.17))
+  (no_connect (at 59.69 85.09))
+  (no_connect (at 85.09 85.09))
+  (wire (pts (xy 67.31 105.41) (xy 67.31 113.03))
     (stroke (width 0) (type default) (color 0 0 0 0))
   )
-  (wire (pts (xy 69.85 105.41) (xy 69.85 111.76))
+  (wire (pts (xy 85.09 69.85) (xy 96.52 69.85))
     (stroke (width 0) (type default) (color 0 0 0 0))
   )
-  (wire (pts (xy 69.85 111.76) (xy 74.93 111.76))
+  (wire (pts (xy 69.85 46.99) (xy 69.85 59.69))
     (stroke (width 0) (type default) (color 0 0 0 0))
   )
@@
     (stroke (width 0) (type default) (color 0 0 0 0))
   )
-  (wire (pts (xy 95.25 87.63) (xy 85.09 87.63))
+  (wire (pts (xy 77.47 105.41) (xy 77.47 113.03))
     (stroke (width 0) (type default) (color 0 0 0 0))
   )
-  (wire (pts (xy 85.09 69.85) (xy 95.25 69.85))
-    (stroke (width 0) (type default) (color 0 0 0 0))
-  )
-  (wire (pts (xy 66.04 111.76) (xy 67.31 111.76))
-    (stroke (width 0) (type default) (color 0 0 0 0))
-  )
-  (wire (pts (xy 85.09 85.09) (xy 95.25 85.09))
-    (stroke (width 0) (type default) (color 0 0 0 0))
-  )
-  (wire (pts (xy 85.09 72.39) (xy 95.25 72.39))
-    (stroke (width 0) (type default) (color 0 0 0 0))
-  )
-  (wire (pts (xy 69.85 46.99) (xy 69.85 59.69))
+  (wire (pts (xy 85.09 74.93) (xy 88.9 74.93))
     (stroke (width 0) (type default) (color 0 0 0 0))
   )
@@
     (stroke (width 0) (type default) (color 0 0 0 0))
   )
-  (wire (pts (xy 67.31 105.41) (xy 67.31 111.76))
+  (wire (pts (xy 88.9 72.39) (xy 96.52 72.39))
     (stroke (width 0) (type default) (color 0 0 0 0))
   )
-  (wire (pts (xy 74.93 111.76) (xy 77.47 111.76))
+  (wire (pts (xy 74.93 113.03) (xy 72.39 113.03))
     (stroke (width 0) (type default) (color 0 0 0 0))
   )
-  (wire (pts (xy 77.47 111.76) (xy 77.47 105.41))
+  (wire (pts (xy 74.93 105.41) (xy 74.93 113.03))
     (stroke (width 0) (type default) (color 0 0 0 0))
   )
-  (wire (pts (xy 85.09 87.63) (xy 85.09 90.17))
+  (wire (pts (xy 72.39 113.03) (xy 72.39 118.11))
     (stroke (width 0) (type default) (color 0 0 0 0))
   )
@@
     (stroke (width 0) (type default) (color 0 0 0 0))
   )
-  (wire (pts (xy 74.93 48.26) (xy 74.93 59.69))
+  (wire (pts (xy 67.31 113.03) (xy 69.85 113.03))
     (stroke (width 0) (type default) (color 0 0 0 0))
   )
-  (wire (pts (xy 85.09 74.93) (xy 85.09 72.39))
+  (wire (pts (xy 72.39 113.03) (xy 69.85 113.03))
     (stroke (width 0) (type default) (color 0 0 0 0))
   )
-  (wire (pts (xy 67.31 111.76) (xy 69.85 111.76))
+  (wire (pts (xy 74.93 45.72) (xy 74.93 59.69))
     (stroke (width 0) (type default) (color 0 0 0 0))
   )
-  (hierarchical_label "+12V" (shape input) (at 74.93 48.26 90)
+  (wire (pts (xy 88.9 74.93) (xy 88.9 72.39))
+    (stroke (width 0) (type default) (color 0 0 0 0))
+  )
+  (wire (pts (xy 69.85 113.03) (xy 69.85 105.41))
+    (stroke (width 0) (type default) (color 0 0 0 0))
+  )
+  (wire (pts (xy 77.47 113.03) (xy 74.93 113.03))
+    (stroke (width 0) (type default) (color 0 0 0 0))
+  )
+  (hierarchical_label "+12V" (shape input) (at 74.93 45.72 90)
     (effects (font (size 1.27 1.27)) (justify left))
+  )
+  (hierarchical_label "GND" (shape input) (at 72.39 118.11 270)
+    (effects (font (size 1.27 1.27)) (justify right))
   )
   (hierarchical_label "MOTOR_DIRECTION_2" (shape input) (at 41.91 74.93 180)
@@
     (effects (font (size 1.27 1.27)) (justify left))
   )
-  (hierarchical_label "GND" (shape input) (at 66.04 111.76 180)
-    (effects (font (size 1.27 1.27)) (justify right))
-  )
   (hierarchical_label "MOTOR_PWM" (shape input) (at 43.18 80.01 180)
     (effects (font (size 1.27 1.27)) (justify right))
@@
     (effects (font (size 1.27 1.27)) (justify right))
   )
-  (symbol (lib_id "Connector_Generic:Conn_01x02") (at 100.33 85.09 0) (unit 1)
+  (symbol (lib_id "Connector_Generic:Conn_01x02") (at 101.6 69.85 0) (unit 1)
     (in_bom yes) (on_board yes) (fields_autoplaced)
-    (property "Reference" "MOTOR2" (id 0) (at 102.87 85.0899 0)
+    (property "Reference" "MOTOR1" (id 0) (at 104.14 69.8499 0)
       (effects (font (size 1.27 1.27)) (justify left))
     )
-    (property "Value" "MOTOR" (id 1) (at 102.87 87.6299 0)
+    (property "Value" "MOTOR" (id 1) (at 104.14 72.3899 0)
       (effects (font (size 1.27 1.27)) (justify left))
     )
-    (property "Footprint" "Connector_PinHeader_2.54mm:PinHeader_1x02_P2.54mm_Vertical" (id 2) (at 100.33 85.09 0)
+    (property "Footprint" "Connector_JST:JST_XH_B2B-XH-A_1x02_P2.50mm_Vertical" (id 2) (at 101.6 69.85 0)
       (effects (font (size 1.27 1.27)) hide)
     )
-    (property "Datasheet" "~" (id 3) (at 100.33 85.09 0)
+    (property "Datasheet" "~" (id 3) (at 101.6 69.85 0)
       (effects (font (size 1.27 1.27)) hide)
     )
@@
   (symbol (lib_id "Driver_Motor:L293D") (at 72.39 85.09 0) (unit 1)
     (in_bom yes) (on_board yes) (fields_autoplaced)
-    (property "Reference" "U3" (id 0) (at 76.9494 57.15 0)
+    (property "Reference" "U2" (id 0) (at 76.9494 57.15 0)
       (effects (font (size 1.27 1.27)) (justify left))
     )
@@
     (pin "9")
   )
-  (symbol (lib_id "Connector_Generic:Conn_01x02") (at 100.33 69.85 0) (unit 1)
-    (in_bom yes) (on_board yes) (fields_autoplaced)
-    (property "Reference" "MOTOR1" (id 0) (at 102.87 69.8499 0)
-      (effects (font (size 1.27 1.27)) (justify left))
-    )
-    (property "Value" "MOTOR" (id 1) (at 102.87 72.3899 0)
-      (effects (font (size 1.27 1.27)) (justify left))
-    )
-    (property "Footprint" "Connector_PinHeader_2.54mm:PinHeader_1x02_P2.54mm_Vertical" (id 2) (at 100.33 69.85 0)
-      (effects (font (size 1.27 1.27)) hide)
-    )
-    (property "Datasheet" "~" (id 3) (at 100.33 69.85 0)
-      (effects (font (size 1.27 1.27)) hide)
-    )
-    (pin "1")
-    (pin "2")
-  )
 )
