File: schematics/sailboard-esp/sailboard-esp.kicad_sch (KiCad schematic)
At the start: 11 parts, among them J2 MainPowerSwitch

Commit message: v1.1 of sailboard.
Parts:
- removed SDCARD1: SD Card, Connector_PinHeader_2.00mm:PinHeader_1x06_P2.00mm_Vertical, symbol Russell:SD Card
- added BATCHRG1: BatteryCharge, Connector_PinHeader_2.00mm:PinHeader_1x02_P2.00mm_Vertical, symbol Connector:Conn_01x02_Male
- added MICRO_SD: Micro_SD_Card, Connector_Card:microSD_HC_Molex_104031-0811, symbol Connector:Micro_SD_Card
- added SOLARIN1: SolarPanel, Connector_PinHeader_2.00mm:PinHeader_1x02_P2.00mm_Vertical, symbol Connector:Conn_01x02_Male
- ArduCam1: footprint Connector_PinHeader_2.00mm:PinHeader_1x08_P2.00mm_Vertical -> Connector_PinHeader_2.54mm:PinHeader_1x08_P2.54mm_Vertical
- COMPASS1: footprint Connector_PinHeader_2.00mm:PinHeader_1x05_P2.00mm_Vertical -> Connector_PinHeader_2.54mm:PinHeader_1x05_P2.54mm_Vertical
- GPS1: footprint Connector_PinHeader_1.00mm:PinHeader_1x04_P1.00mm_Vertical -> Connector_PinHeader_2.54mm:PinHeader_1x04_P2.54mm_Vertical
- renumbered J2 to MAINSWITCH1
Connections:
- net +3.3V: now also MICRO_SD.4 (VDD)
- net GND: now also MICRO_SD.6 (VSS)
- net MISO: now also MICRO_SD.3 (CMD)
- net MOSI: now also MICRO_SD.7 (DAT0)
- net SCK: now also MICRO_SD.5 (CLK)
- net SDCARD_CS: now also MICRO_SD.2 (DAT3/CD)
- new net Power/Battery Charge Neg: BATCHRG1.2 (Pin_2)
- new net Power/Battery Charge Pos: BATCHRG1.1 (Pin_1)
- new net Power/Solar Neg: SOLARIN1.2 (Pin_2)
- new net Power/Solar Pos: SOLARIN1.1 (Pin_1)
- no-connect marks 5 -> 8
Other:
- sheet Power ports: added Battery Charge Neg, Battery Charge Pos, Solar Neg, Solar Pos; removed none

Commit message: version 1.1.
Parts:
- BATCHRG1, BATIN1, MAINSWITCH1, SOLARIN1: footprint Connector_PinHeader_2.00mm:PinHeader_1x02_P2.00mm_Vertical -> Connector_PinHeader_2.54mm:PinHeader_1x02_P2.54mm_Vertical
- D2: footprint LED_SMD:LED_0402_1005Metric -> LED_SMD:LED_0603_1608Metric
- RUDDER1: footprint Connector_PinHeader_2.00mm:PinHeader_1x03_P2.00mm_Vertical -> Connector_PinHeader_2.54mm:PinHeader_1x03_P2.54mm_Vertical
- renumbered MICRO_SD to MICRO_SD1
Connections:
- net +3.3V: now also R1.1
- net +5V: no longer R1.1
Changed lines of the file:
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@@
     (property "Reference" "MAINSWITCH1" (id 0) (at 22.225 36.83 0))
     (property "Value" "MainPowerSwitch" (id 1) (at 22.225 39.37 0))
-    (property "Footprint" "Connector_PinHeader_2.00mm:PinHeader_1x02_P2.00mm_Vertical" (id 2) (at 21.59 41.91 0)
+    (property "Footprint" "Connector_PinHeader_2.54mm:PinHeader_1x02_P2.54mm_Vertical" (id 2) (at 21.59 41.91 0)
       (effects (font (size 1.27 1.27)) hide)
     )
@@
     (property "Reference" "BATIN1" (id 0) (at 22.225 22.86 0))
     (property "Value" "BatteryInput" (id 1) (at 20.32 26.67 0))
-    (property "Footprint" "Connector_PinHeader_2.00mm:PinHeader_1x02_P2.00mm_Vertical" (id 2) (at 21.59 27.94 0)
+    (property "Footprint" "Connector_PinHeader_2.54mm:PinHeader_1x02_P2.54mm_Vertical" (id 2) (at 21.59 27.94 0)
       (effects (font (size 1.27 1.27)) hide)
     )
@@
       (effects (font (size 1.27 1.27)) (justify left))
     )
-    (property "Footprint" "Connector_PinHeader_2.00mm:PinHeader_1x03_P2.00mm_Vertical" (id 2) (at 177.8 121.92 0)
+    (property "Footprint" "Connector_PinHeader_2.54mm:PinHeader_1x03_P2.54mm_Vertical" (id 2) (at 177.8 121.92 0)
       (effects (font (size 1.27 1.27)) hide)
     )
@@
     )
     (property "Datasheet" "" (id 3) (at 45.72 120.65 0)
-      (effects (font (size 1.27 1.27)) hide)
-    )
-    (pin "1")
-  )
-  (symbol (lib_id "power:+5V") (at 21.59 78.74 0) (unit 1)
-    (in_bom yes) (on_board yes) (fields_autoplaced)
-    (property "Reference" "#PWR0136" (id 0) (at 21.59 82.55 0)
-      (effects (font (size 1.27 1.27)) hide)
-    )
-    (property "Value" "+5V" (id 1) (at 21.59 73.66 0))
-    (property "Footprint" "" (id 2) (at 21.59 78.74 0)
-      (effects (font (size 1.27 1.27)) hide)
-    )
-    (property "Datasheet" "" (id 3) (at 21.59 78.74 0)
       (effects (font (size 1.27 1.27)) hide)
     )
@@
     (property "Reference" "SOLARIN1" (id 0) (at 22.225 48.26 0))
     (property "Value" "SolarPanel" (id 1) (at 20.32 52.07 0))
-    (property "Footprint" "Connector_PinHeader_2.00mm:PinHeader_1x02_P2.00mm_Vertical" (id 2) (at 21.59 53.34 0)
+    (property "Footprint" "Connector_PinHeader_2.54mm:PinHeader_1x02_P2.54mm_Vertical" (id 2) (at 21.59 53.34 0)
       (effects (font (size 1.27 1.27)) hide)
     )
@@
     (pin "1")
   )
+  (symbol (lib_id "power:+3.3V") (at 21.59 78.74 0) (unit 1)
+    (in_bom yes) (on_board yes) (fields_autoplaced)
+    (property "Reference" "#PWR0136" (id 0) (at 21.59 82.55 0)
+      (effects (font (size 1.27 1.27)) hide)
+    )
+    (property "Value" "+3.3V" (id 1) (at 21.59 73.66 0))
+    (property "Footprint" "" (id 2) (at 21.59 78.74 0)
+      (effects (font (size 1.27 1.27)) hide)
+    )
+    (property "Datasheet" "" (id 3) (at 21.59 78.74 0)
+      (effects (font (size 1.27 1.27)) hide)
+    )
+    (pin "1")
+  )
   (symbol (lib_id "Device:LED") (at 45.72 81.28 180) (unit 1)
     (in_bom yes) (on_board yes) (fields_autoplaced)
     (property "Reference" "D2" (id 0) (at 47.3075 73.66 0))
     (property "Value" "LED" (id 1) (at 47.3075 76.2 0))
-    (property "Footprint" "LED_SMD:LED_0402_1005Metric" (id 2) (at 45.72 81.28 0)
+    (property "Footprint" "LED_SMD:LED_0603_1608Metric" (id 2) (at 45.72 81.28 0)
       (effects (font (size 1.27 1.27)) hide)
     )
@@
     (property "Reference" "BATCHRG1" (id 0) (at 15.24 62.23 0))
     (property "Value" "BatteryCharge" (id 1) (at 21.59 59.69 0))
-    (property "Footprint" "Connector_PinHeader_2.00mm:PinHeader_1x02_P2.00mm_Vertical" (id 2) (at 22.86 60.96 0)
+    (property "Footprint" "Connector_PinHeader_2.54mm:PinHeader_1x02_P2.54mm_Vertical" (id 2) (at 22.86 60.96 0)
       (effects (font (size 1.27 1.27)) hide)
     )
@@
   (symbol (lib_id "Connector:Micro_SD_Card") (at 259.08 104.14 0) (unit 1)
     (in_bom yes) (on_board yes) (fields_autoplaced)
-    (property "Reference" "MICRO_SD" (id 0) (at 259.715 85.09 0))
+    (property "Reference" "MICRO_SD1" (id 0) (at 259.715 85.09 0))
     (property "Value" "Micro_SD_Card" (id 1) (at 259.715 87.63 0))
     (property "Footprint" "Connector_Card:microSD_HC_Molex_104031-0811" (id 2) (at 288.29 96.52 0)
@@
       (reference "#PWR0108") (unit 1) (value "GND") (footprint "")
     )
-    (path "/646f8b99-5d19-4d75-969e-577fa29dc718/35677b2a-3255-4ee6-8e26-f36f61954655"
-      (reference "#PWR0109") (unit 1) (value "+5V") (footprint "")
+    (path "/646f8b99-5d19-4d75-969e-577fa29dc718/c3f20993-703b-4ef4-a2a5-e61dca408474"
+      (reference "#PWR0109") (unit 1) (value "+3.3V") (footprint "")
     )
     (path "/646f8b99-5d19-4d75-969e-577fa29dc718/f7426d7a-e06c-4520-adcd-836ef3b8416b"
@@
       (reference "#PWR0135") (unit 1) (value "GND") (footprint "")
     )
-    (path "/4a93f704-d5cb-4204-99a5-99ad240b4b5a"
-      (reference "#PWR0136") (unit 1) (value "+5V") (footprint "")
+    (path "/af6fffb2-814c-4fce-935e-cd253dd7e2aa"
+      (reference "#PWR0136") (unit 1) (value "+3.3V") (footprint "")
     )
     (path "/d800a68a-b097-4844-953b-f506858f898f"
@@
       (reference "#PWR0147") (unit 1) (value "GND") (footprint "")
     )
-    (path "/646f8b99-5d19-4d75-969e-577fa29dc718/23609877-3dea-4d8c-97b2-a43bc284cf08"
-      (reference "#PWR0148") (unit 1) (value "+5V") (footprint "")
+    (path "/646f8b99-5d19-4d75-969e-577fa29dc718/8304e128-fcea-43b3-b9b8-b49217930df6"
+      (reference "#PWR0148") (unit 1) (value "+3.3V") (footprint "")
     )
     (path "/646f8b99-5d19-4d75-969e-577fa29dc718/7dfeb57d-6fe3-4f4a-b407-904970e5d564"
       (reference "#PWR0149") (unit 1) (value "GND") (footprint "")
     )
-    (path "/646f8b99-5d19-4d75-969e-577fa29dc718/96db91c8-5540-4330-a0a3-a518871f9f86"
-      (reference "#PWR0150") (unit 1) (value "+5V") (footprint "")
+    (path "/646f8b99-5d19-4d75-969e-577fa29dc718/4c28b569-cef3-40ae-80a8-53ad3246cbfa"
+      (reference "#PWR0150") (unit 1) (value "+3.3V") (footprint "")
     )
     (path "/646f8b99-5d19-4d75-969e-577fa29dc718/57c11d52-356a-42e8-b462-e55f52cb62b4"
       (reference "#PWR0151") (unit 1) (value "GND") (footprint "")
     )
-    (path "/646f8b99-5d19-4d75-969e-577fa29dc718/644f6e85-dd1d-4b1c-ba3d-18e75e67a517"
-      (reference "#PWR0152") (unit 1) (value "+5V") (footprint "")
-    )
     (path "/7a85f1c8-4b71-41a9-8803-d105b98e9320/833461f6-8bad-4cce-a8a6-2e7557987be6"
       (reference "#PWR0153") (unit 1) (value "+3.3V") (footprint "")
@@
     )
     (path "/b265728d-a538-4111-9e95-1b5dc4d0bf65"
-      (reference "BATCHRG1") (unit 1) (value "BatteryCharge") (footprint "Connector_PinHeader_2.00mm:PinHeader_1x02_P2.00mm_Vertical")
+      (reference "BATCHRG1") (unit 1) (value "BatteryCharge") (footprint "Connector_PinHeader_2.54mm:PinHeader_1x02_P2.54mm_Vertical")
     )
     (path "/20e4f168-b2ff-4be5-8df9-c3aa2255b665"
-      (reference "BATIN1") (unit 1) (value "BatteryInput") (footprint "Connector_PinHeader_2.00mm:PinHeader_1x02_P2.00mm_Vertical")
+      (reference "BATIN1") (unit 1) (value "BatteryInput") (footprint "Connector_PinHeader_2.54mm:PinHeader_1x02_P2.54mm_Vertical")
     )
     (path "/646f8b99-5d19-4d75-969e-577fa29dc718/51c45aa0-32bb-466f-ad0a-8fa67626b138"
@@
     )
     (path "/b0e566c3-0469-4470-8762-aa348871e5ef"
-      (reference "D2") (unit 1) (value "LED") (footprint "LED_SMD:LED_0402_1005Metric")
+      (reference "D2") (unit 1) (value "LED") (footprint "LED_SMD:LED_0603_1608Metric")
     )
     (path "/7a85f1c8-4b71-41a9-8803-d105b98e9320/4940d571-7598-442c-bd21-1a8a4a260dc6"
@@
     )
     (path "/1c32450b-32f4-4dca-8cd7-fa69196d822e"
-      (reference "MAINSWITCH1") (unit 1) (value "MainPowerSwitch") (footprint "Connector_PinHeader_2.00mm:PinHeader_1x02_P2.00mm_Vertical")
+      (reference "MAINSWITCH1") (unit 1) (value "MainPowerSwitch") (footprint "Connector_PinHeader_2.54mm:PinHeader_1x02_P2.54mm_Vertical")
     )
     (path "/c0826052-1270-4dc8-967d-3ccc9bc5794a"
-      (reference "MICRO_SD") (unit 1) (value "Micro_SD_Card") (footprint "Connector_Card:microSD_HC_Molex_104031-0811")
+      (reference "MICRO_SD1") (unit 1) (value "Micro_SD_Card") (footprint "Connector_Card:microSD_HC_Molex_104031-0811")
     )
     (path "/96f7984a-83d5-40aa-b38c-0b027701a1c8/e041920d-b43c-4909-bb86-f3181b925256"
-      (reference "MOTOR1") (unit 1) (value "MOTOR") (footprint "Connector_PinHeader_2.00mm:PinHeader_1x02_P2.00mm_Vertical")
+      (reference "MOTOR1") (unit 1) (value "MOTOR") (footprint "Connector_PinHeader_2.54mm:PinHeader_1x02_P2.54mm_Vertical")
     )
     (path "/96f7984a-83d5-40aa-b38c-0b027701a1c8/4e61bf96-81b2-466e-b245-17b998b919c6"
-      (reference "MOTOR2") (unit 1) (value "MOTOR") (footprint "Connector_PinHeader_2.00mm:PinHeader_1x02_P2.00mm_Vertical")
+      (reference "MOTOR2") (unit 1) (value "MOTOR") (footprint "Connector_PinHeader_2.54mm:PinHeader_1x02_P2.54mm_Vertical")
     )
     (path "/b502c931-5fd6-463b-a803-b08a5926f599"
@@
     )
     (path "/233f1ce8-fd0b-448f-8d1b-84d4d750d93f"
-      (reference "RUDDER1") (unit 1) (value "RUDDERSERVO") (footprint "Connector_PinHeader_2.00mm:PinHeader_1x03_P2.00mm_Vertical")
+      (reference "RUDDER1") (unit 1) (value "RUDDERSERVO") (footprint "Connector_PinHeader_2.54mm:PinHeader_1x03_P2.54mm_Vertical")
     )
     (path "/646f8b99-5d19-4d75-969e-577fa29dc718/a9654ecd-7c40-4441-a656-9e905467f463"
@@
     )
     (path "/6a262e40-15f4-4bfc-b575-39ef2f86d95f"
-      (reference "SOLARIN1") (unit 1) (value "SolarPanel") (footprint "Connector_PinHeader_2.00mm:PinHeader_1x02_P2.00mm_Vertical")
+      (reference "SOLARIN1") (unit 1) (value "SolarPanel") (footprint "Connector_PinHeader_2.54mm:PinHeader_1x02_P2.54mm_Vertical")
     )
     (path "/96f7984a-83d5-40aa-b38c-0b027701a1c8/b9fd611f-b8fa-4bd1-98bd-f9a1bb7af07a"

Commit message: move to version 1.2.
Parts:
- BATCHRG1, BATIN1, MAINSWITCH1, SOLARIN1: footprint Connector_PinHeader_2.54mm:PinHeader_1x02_P2.54mm_Vertical -> Connector_JST:JST_XH_B2B-XH-A_1x02_P2.50mm_Vertical
- RUDDER1: footprint Connector_PinHeader_2.54mm:PinHeader_1x03_P2.54mm_Vertical -> Connector_JST:JST_XH_B3B-XH-A_1x03_P2.50mm_Vertical
Connections:
- net MISO: no longer MICRO_SD1.3 (CMD)
- net MOSI: no longer MICRO_SD1.7 (DAT0)
- net SCK: no longer MICRO_SD1.5 (CLK)
- net SDCARD_CS: no longer MICRO_SD1.2 (DAT3/CD)
- net SDCARD_D2: now reaches MICRO_SD1.1 (DAT2)
- net SDCARD_D1: now reaches MICRO_SD1.8 (DAT1)
- net CS renamed ARDUCAM_CS
- new net SDCARD_CMD: MICRO_SD1.3 (CMD)
- new net SDCARD_D0: MICRO_SD1.7 (DAT0)
- new net SDCARD_D3: MICRO_SD1.2 (DAT3/CD)
- new net SDCARD_SCK: MICRO_SD1.5 (CLK)
- no-connect marks 8 -> 5
Other:
- sheet Microcontroller ports: added ARDUCAM_CS, SDCARD_CMD, SDCARD_CS, SDCARD_D0, SDCARD_D1, SDCARD_D2, SDCARD_D3, SDCARD_SCK; removed none

Commit message: added changelog and tweaks.
Parts:
- added C4: 470uF, Capacitor_THT:CP_Radial_D8.0mm_P3.50mm, symbol Device:C_Polarized_Small_US
Connections:
- net +5V: now also C4.1
- net GND: now also C4.2
Changed lines of the file:
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@@
     (rev "v1")
+  )
+  (junction (at 157.48 118.11) (diameter 0) (color 0 0 0 0)
+  )
+  (junction (at 167.64 118.11) (diameter 0) (color 0 0 0 0)
   )
   (no_connect (at 171.45 140.97))
@@
     (stroke (width 0) (type default) (color 0 0 0 0))
   )
+  (wire (pts (xy 157.48 118.11) (xy 160.02 118.11))
+    (stroke (width 0) (type default) (color 0 0 0 0))
+  )
   (wire (pts (xy 50.8 39.37) (xy 53.34 39.37))
     (stroke (width 0) (type default) (color 0 0 0 0))
@@
     (stroke (width 0) (type default) (color 0 0 0 0))
   )
+  (wire (pts (xy 157.48 118.11) (xy 157.48 116.84))
+    (stroke (width 0) (type default) (color 0 0 0 0))
+  )
   (wire (pts (xy 231.14 31.75) (xy 231.14 52.07))
     (stroke (width 0) (type default) (color 0 0 0 0))
@@
     (stroke (width 0) (type default) (color 0 0 0 0))
   )
-  (wire (pts (xy 172.72 121.92) (xy 162.56 121.92))
+  (wire (pts (xy 172.72 121.92) (xy 157.48 121.92))
     (stroke (width 0) (type default) (color 0 0 0 0))
   )
@@
     (stroke (width 0) (type default) (color 0 0 0 0))
   )
-  (wire (pts (xy 167.64 115.57) (xy 167.64 119.38))
+  (wire (pts (xy 167.64 115.57) (xy 167.64 118.11))
+    (stroke (width 0) (type default) (color 0 0 0 0))
+  )
+  (wire (pts (xy 167.64 118.11) (xy 167.64 119.38))
     (stroke (width 0) (type default) (color 0 0 0 0))
   )
@@
     (stroke (width 0) (type default) (color 0 0 0 0))
   )
-  (wire (pts (xy 162.56 121.92) (xy 162.56 116.84))
+  (wire (pts (xy 157.48 121.92) (xy 157.48 118.11))
     (stroke (width 0) (type default) (color 0 0 0 0))
   )
@@
   )
   (wire (pts (xy 215.9 104.14) (xy 236.22 104.14))
+    (stroke (width 0) (type default) (color 0 0 0 0))
+  )
+  (wire (pts (xy 165.1 118.11) (xy 167.64 118.11))
     (stroke (width 0) (type default) (color 0 0 0 0))
   )
@@
     (pin "3")
   )
+  (symbol (lib_id "Device:C_Polarized_Small_US") (at 162.56 118.11 270) (unit 1)
+    (in_bom yes) (on_board yes) (fields_autoplaced)
+    (property "Reference" "C4" (id 0) (at 162.9918 111.76 90))
+    (property "Value" "470uF" (id 1) (at 162.9918 114.3 90))
+    (property "Footprint" "Capacitor_THT:CP_Radial_D8.0mm_P3.50mm" (id 2) (at 162.56 118.11 0)
+      (effects (font (size 1.27 1.27)) hide)
+    )
+    (property "Datasheet" "~" (id 3) (at 162.56 118.11 0)
+      (effects (font (size 1.27 1.27)) hide)
+    )
+    (pin "1")
+    (pin "2")
+  )
   (symbol (lib_id "power:GND") (at 54.61 81.28 90) (unit 1)
     (in_bom yes) (on_board yes) (fields_autoplaced)
@@
     (pin "1")
   )
-  (symbol (lib_id "power:GND") (at 162.56 116.84 180) (unit 1)
-    (in_bom yes) (on_board yes) (fields_autoplaced)
-    (property "Reference" "#PWR0133" (id 0) (at 162.56 110.49 0)
-      (effects (font (size 1.27 1.27)) hide)
-    )
-    (property "Value" "GND" (id 1) (at 162.56 111.76 0))
-    (property "Footprint" "" (id 2) (at 162.56 116.84 0)
-      (effects (font (size 1.27 1.27)) hide)
-    )
-    (property "Datasheet" "" (id 3) (at 162.56 116.84 0)
+  (symbol (lib_id "power:GND") (at 157.48 116.84 180) (unit 1)
+    (in_bom yes) (on_board yes) (fields_autoplaced)
+    (property "Reference" "#PWR0133" (id 0) (at 157.48 110.49 0)
+      (effects (font (size 1.27 1.27)) hide)
+    )
+    (property "Value" "GND" (id 1) (at 157.48 111.76 0))
+    (property "Footprint" "" (id 2) (at 157.48 116.84 0)
+      (effects (font (size 1.27 1.27)) hide)
+    )
+    (property "Datasheet" "" (id 3) (at 157.48 116.84 0)
       (effects (font (size 1.27 1.27)) hide)
     )
@@
       (reference "C3") (unit 1) (value "22uF") (footprint "Capacitor_SMD:C_0603_1608Metric_Pad1.08x0.95mm_HandSolder")
     )
+    (path "/24edccf9-c8a4-48a1-a5d9-88f54743e392"
+      (reference "C4") (unit 1) (value "470uF") (footprint "Capacitor_THT:CP_Radial_D8.0mm_P3.50mm")
+    )
     (path "/1cd4d1a3-45f5-417d-b61e-2caadbb9fed8"

Commit message: v1.3.
Parts:
- added R6, R7: 47K ARRAY, RESCAXE80P320X160X70-8N, symbol YC164-JR-0747KL:YC164-JR-0747KL
Connections:
- net +3.3V: now also COMPASS1.1 (VCC), R6.6, R6.7, R6.8, R7.1, R7.2, R7.3, R7.4; no longer COMPASS1.2 (VCC)
- net +5V: now also IRIDIUM1.3 (5V); no longer IRIDIUM1.8 (5V)
- net GND: now also COMPASS1.2 (GND), IRIDIUM1.1 (GND); no longer COMPASS1.1 (GND), IRIDIUM1.10 (GND)
- net IRIDIUM_RING: now also IRIDIUM1.6 (RING); no longer IRIDIUM1.5 (RING)
- net IRIDIUM_RX: now also IRIDIUM1.10 (RXD); no longer IRIDIUM1.1 (RXD)
- net IRIDIUM_SLEEP: now also IRIDIUM1.4 (SLEEP); no longer IRIDIUM1.7 (SLEEP)
- net IRIDIUM_TX: now also IRIDIUM1.5 (TXD); no longer IRIDIUM1.6 (TXD)
- net SDCARD_CMD: now also R6.2
- net SDCARD_D0: now also R7.7
- net SDCARD_D1: now also R7.8
- net SDCARD_D2: now also R6.4
- net SDCARD_D3: now also R6.3
- net SDCARD_SCK: now also R7.6
Other:
- moved on the sheet: ArduCam1, C4, COMPASS1, GPS1, IRIDIUM1, RUDDER1
